Commit message: Finished URDF for block robot arm

File: clam_description/urdf/materials.urdf.xacro (robot description, xacro)
@@ -7,6 +7,6 @@
         <color rgba="0.0 0.0 0.8 1.0"/>
     </material>
-    <material name="Orange">
-        <color rgba="183 94 32 1.0"/>
+    <material name="Green">
+        <color rgba="0.0 0.8 0.0 1.0"/>
     </material>
     <material name="Grey">

Commit message: Converted all names to 'clam'

File: clam_description/urdf/materials.urdf.xacro (robot description, xacro)
@@ -22,6 +22,6 @@
         <color rgba="1.0 1.0 1.0 1.0"/>
     </material>
-    <material name="GunMetalBrushedAluminum">
+    <!--material name="GunMetalBrushedAluminum">
         <texture filename="package://smart_arm_description/Media/materials/textures/gun_metal_brushed_aluminum.jpg" />
-    </material>
+    </material-->
 </robot>

Commit message: Created rough 3d visulization

File: clam_description/urdf/materials.urdf.xacro (robot description, xacro)
@@ -22,6 +22,6 @@
         <color rgba="1.0 1.0 1.0 1.0"/>
     </material>
-    <!--material name="GunMetalBrushedAluminum">
-        <texture filename="package://smart_arm_description/Media/materials/textures/gun_metal_brushed_aluminum.jpg" />
-    </material-->
+    <material name="GunMetalBrushedAluminum">
+        <texture filename="package://clam_description/media/gun_metal_brushed_aluminum.jpg" />
+    </material>
 </robot>

Commit message: Updated arm naivgation

File: clam_description/urdf/materials.urdf.xacro (robot description, xacro)
@@ -2,5 +2,5 @@
 <robot>
     <material name="Black">
-        <color rgba="0.1 0.0 0.0 1.0"/>
+        <color rgba="0.0 0.0 0.0 1.0"/>
     </material>
     <material name="Blue">
@@ -11,8 +11,8 @@
     </material>
     <material name="Grey">
-        <color rgba="0.7 0.7 0.7 1.0"/>
+        <color rgba="0.2 0.2 0.2 1.0"/>
     </material>
-    <material name="Grey2">
-        <color rgba="0.9 0.9 0.9 1.0"/>
+    <material name="Orange">
+        <color rgba="${255/255} ${108/255} ${10/255} 1.0"/>
     </material>
     <material name="Red">
