Commit message: Integrating new clam cad models into urdf

File: clam_description/urdf/clam_urdf_andy.urdf (robot description, URDF)
Before this commit: robot clam, 7 links, 6 joints
Links:
- added link gripper_roll_link; visual mesh filename=package://clam_description/stl/gripper_grip_link.STL scale=0.001 0.001 0.001
- added link l_gripper_aft_link; visual mesh filename=package://clam_description/stl/l_gripper_aft_link.STL scale=0.001 0.001 0.001
- added link l_gripper_fwd_link; visual mesh filename=package://clam_description/stl/l_gripper_fwd_link.STL scale=0.001 0.001 0.001
- added link l_gripper_pincher; visual mesh filename=package://clam_description/stl/l_gripper_pincher.STL scale=0.001 0.001 0.001
- added link r_gripper_aft_link; visual mesh filename=package://clam_description/stl/r_gripper_aft_link.STL scale=0.001 0.001 0.001
- added link r_gripper_fwd_link; visual mesh filename=package://clam_description/stl/r_gripper_fwd_link.STL scale=0.001 0.001 0.001
- added link r_gripper_pincher; visual mesh filename=package://clam_description/stl/r_gripper_pincher.STL scale=0.001 0.001 0.001
Joints:
- added joint gripper_roll_joint: type revolute, parent wrist_pitch_link, child gripper_roll_link, origin xyz=0 0 0.08 rpy=0 -1.570795 0, axis 1 0 0, limit lower=-2.61799387799 upper=2.6128806087 effort=300 velocity=1
- added joint l_gripper_aft_link_joint: type revolute, parent gripper_roll_link, child l_gripper_aft_link, origin xyz=0.025 -0.0275 0 rpy=0 -1.570795 0.603534345556, axis 1 0 0, limit lower=0.0 upper=0.925023722222 effort=300 velocity=1
- added joint l_gripper_aft_pincher_joint: type continuous, parent l_gripper_aft_link, child l_gripper_pincher, origin xyz=0.0032 0 -0.0508 rpy=3.54772777389 0 0, axis 1 0 0, limit lower=-1.57 upper=1.57 effort=300 velocity=1, mimic joint=l_gripper_aft_link_joint multiplier=-1.0 offset=0
- added joint l_gripper_fwd_link_joint: type revolute, parent gripper_roll_link, child l_gripper_fwd_link, origin xyz=0.05 -0.037 0.007 rpy=0 -1.570795 3.74512434556, axis 1 0 0, limit lower=0 upper=1.57 effort=300 velocity=1, mimic joint=l_gripper_aft_link_joint multiplier=1.0 offset=0
- added joint r_gripper_aft_link_joint: type revolute, parent gripper_roll_link, child r_gripper_aft_link, origin xyz=0.025 -0.0561 0 rpy=0 -1.570795 -0.603534345556, axis 1 0 0, limit lower=-3.14 upper=3.14 effort=300 velocity=1, mimic joint=l_gripper_aft_link_joint multiplier=-1.0 offset=0.0
- added joint r_gripper_aft_pincher_joint: type revolute, parent r_gripper_aft_link, child r_gripper_pincher, origin xyz=0 0 -0.0508 rpy=0.406137773889 3.14159 0, axis 1 0 0, limit lower=0 upper=0.01 effort=300 velocity=1, mimic joint=l_gripper_aft_link_joint multiplier=-1.0 offset=0
- added joint r_gripper_fwd_link_joint: type revolute, parent gripper_roll_link, child r_gripper_fwd_link, origin xyz=0.05 -0.047 0.007 rpy=0 -1.570795 2.53805565444, axis 1 0 0, limit lower=-1.57 upper=0 effort=300 velocity=1, mimic joint=l_gripper_aft_link_joint multiplier=-1.0 offset=0
