Commit message: Fixed gripper_grip_link

File: clam_description/urdf/clam_urdf_andy.xacro (robot description, xacro)
@@ -1,18 +1,18 @@
 <?xml version="1.0"?>
 <!-- Robot Description format of CLAM arm
-Dave Coleman - davetcoleman@gmail.com
-1/10/2012
-Documentation:
-URDF
-http://www.ros.org/wiki/urdf/XML
-Joint Safety Limits
-http://www.ros.org/wiki/pr2_controller_manager/safety_limits
-XARCO - Macro Language
-http://www.ros.org/wiki/xacro
+     Dave Coleman - davetcoleman@gmail.com
+     1/10/2012
+     Documentation:
+     URDF
+     http://www.ros.org/wiki/urdf/XML
+     Joint Safety Limits
+     http://www.ros.org/wiki/pr2_controller_manager/safety_limits
+     XARCO - Macro Language
+     http://www.ros.org/wiki/xacro
 -->
 <robot name="clam"
-       xmlns:sensor="http://playerstage.sourceforge.net/gazebo/xmlschema/#sensor"
-       xmlns:controller="http://playerstage.sourceforge.net/gazebo/xmlschema/#controller"
-       xmlns:interface="http://playerstage.sourceforge.net/gazebo/xmlschema/#interface">
+    xmlns:sensor="http://playerstage.sourceforge.net/gazebo/xmlschema/#sensor"
+    xmlns:controller="http://playerstage.sourceforge.net/gazebo/xmlschema/#controller"
+    xmlns:interface="http://playerstage.sourceforge.net/gazebo/xmlschema/#interface">
   <!-- Include materials -->
   <include filename="$(find clam_description)/urdf/materials.urdf.xacro" />
@@ -34,9 +34,9 @@
 	<mesh filename="package://clam_description/stl/base_link_simple.STL" scale="${M_SCALE}" />
       </geometry>
-      </collision>>
-      <inertial>
-	<mass value="25" />
-	<inertia ixx="1.0" ixy ="0.0" ixz="0.0" iyy="1.0" iyz="0.0" izz="1.0" />
-      </inertial>
+    </collision>>
+    <inertial>
+      <mass value="25" />
+      <inertia ixx="1.0" ixy ="0.0" ixz="0.0" iyy="1.0" iyz="0.0" izz="1.0" />
+    </inertial>
   </link>
   <joint name="shoulder_pan_joint" type="revolute">
@@ -201,9 +201,15 @@
       <material name="Orange" />
     </visual>
+    <collision>
+      <origin xyz="0 0 0" rpy="0 0 0" />
+      <geometry>
+	<mesh filename="package://clam_description/stl/gripper_grip_link.STL" scale="1 1 1" />
+      </geometry>
+    </collision>
   </link>
   <joint name="l_gripper_aft_link_joint" type="revolute">
     <parent link="gripper_roll_link"/>
     <child link="l_gripper_aft_link"/>
-    <origin xyz="0.025 ${-0.0275+.040} 0" rpy="0 -${M_PI/2} ${34.58*M_PI/180}" />
+    <origin xyz="0.025 0.0169 0" rpy="0 -${M_PI/2} ${34.58*M_PI/180}" />
     <axis xyz="1 0 0" />
     <limit effort="300" velocity="1" lower="${0*M_PI/180}" upper="${53*M_PI/180}" />
@@ -213,5 +219,5 @@
     <parent link="gripper_roll_link"/>
     <child link="r_gripper_aft_link"/>
-    <origin xyz="0.025 ${-0.0561+.040}  0" rpy="0 -${M_PI/2} ${-34.58*M_PI/180}" />
+    <origin xyz="0.025 -0.0117 0" rpy="0 -${M_PI/2} ${-34.58*M_PI/180}" />
     <axis xyz="1 0 0" />
     <limit effort="300" velocity="1" lower="-3.14" upper="3.14" />
@@ -222,5 +228,5 @@
     <parent link="gripper_roll_link"/>
     <child link="l_gripper_fwd_link"/>
-    <origin xyz="0.05 ${-0.037+.040} 0.007" rpy="0 -${M_PI/2} ${214.58*M_PI/180}" />
+    <origin xyz="0.05 0.0074 0.007" rpy="0 -${M_PI/2} ${214.58*M_PI/180}" />
     <axis xyz="1 0 0" />
     <limit effort="300" velocity="1" lower="0" upper="1.57" />
@@ -231,5 +237,5 @@
     <parent link="gripper_roll_link"/>
     <child link="r_gripper_fwd_link"/>
-    <origin xyz="0.05 ${-0.047+.040} 0.007" rpy="0 -${M_PI/2} ${145.42*M_PI/180}" />
+    <origin xyz="0.05 -0.0026 0.007" rpy="0 -${M_PI/2} ${145.42*M_PI/180}" />
     <axis xyz="1 0 0" />
     <limit effort="300" velocity="1" lower="-1.57" upper="0" />
@@ -242,8 +248,14 @@
       <origin xyz="0 0 0" rpy="0 0 0" />
       <geometry>
-	<mesh filename="package://clam_description/stl/l_gripper_fwd_link.STL" scale="${M_SCALE}" />
-      </geometry>
-      <material name="Grey" />
-    </visual>
+	<mesh filename="package://clam_description/stl/l_gripper_fwd_link.STL" scale="1 1 1" />
+      </geometry>
+      <material name="Grey" />
+    </visual>
+    <collision>
+      <origin xyz="0 0 0" rpy="0 0 0" />
+      <geometry>
+	<mesh filename="package://clam_description/stl/l_gripper_fwd_lik.STL" scale="1 1 1" />
+      </geometry>
+    </collision>
   </link>
   <!-- RIGHT GRIPPER FWD LINK -->
@@ -252,8 +264,14 @@
       <origin xyz="0 0 0" rpy="0 0 0" />
       <geometry>
-	<mesh filename="package://clam_description/stl/r_gripper_fwd_link.STL" scale="${M_SCALE}" />
-      </geometry>
-      <material name="Grey" />
-    </visual>
+	<mesh filename="package://clam_description/stl/r_gripper_fwd_link.STL" scale="1 1 1" />
+      </geometry>
+      <material name="Grey" />
+    </visual>
+    <collision>
+      <origin xyz="0 0 0" rpy="0 0 0" />
+      <geometry>
+	<mesh filename="package://clam_description/stl/r_gripper_fwd_link.STL" scale="1 1 1" />
+      </geometry>
+    </collision>
   </link>
   <!-- LEFT GRIPPER AFT LINK -->
@@ -262,8 +280,14 @@
       <origin xyz="0 0 0" rpy="0 0 0" />
       <geometry>
-	<mesh filename="package://clam_description/stl/l_gripper_aft_link.STL" scale="${M_SCALE}" />
-      </geometry>
-      <material name="Grey" />
-    </visual>
+	<mesh filename="package://clam_description/stl/l_gripper_aft_link.STL" scale="1 1 1" />
+      </geometry>
+      <material name="Grey" />
+    </visual>
+    <collision>
+      <origin xyz="0 0 0" rpy="0 0 0" />
+      <geometry>
+	<mesh filename="package://clam_description/stlf/l_gripper_aft_link.STL" scale="1 1 1" />
+      </geometry>
+    </collision>
   </link>
   <joint name="l_gripper_aft_pincher_joint" type="continuous">
@@ -281,8 +305,14 @@
       <origin xyz="0 0 0" rpy="0 0 0" />
       <geometry>
-	<mesh filename="package://clam_description/stl/r_gripper_aft_link.STL" scale="${M_SCALE}" />
-      </geometry>
-      <material name="Grey" />
-    </visual>
+	<mesh filename="package://clam_description/stl/r_gripper_aft_link.STL" scale="1 1 1" />
+      </geometry>
+      <material name="Grey" />
+    </visual>
+    <collision>
+      <origin xyz="0 0 0" rpy="0 0 0" />
+      <geometry>
+	<mesh filename="package://clam_description/stl/r_gripper_aft_link.STL" scale="1 1 1" />
+      </geometry>
+    </collision>
   </link>
   <joint name="r_gripper_aft_pincher_joint" type="revolute">
@@ -291,27 +321,39 @@
     <origin xyz="0 0 -0.0508" rpy="${23.27*M_PI/180} ${M_PI} 0" />
     <axis xyz="1 0 0" />
-    <limit effort="300" velocity="1" lower="0" upper="1.57" />
+    <limit effort="300" velocity="1" lower="0" upper="0.01" />
     <mimic joint="l_gripper_aft_link_joint" multiplier="-1.0" offset="0" />
     <dynamics damping="50" friction="1"/>
   </joint>
-  <!-- LEFT GRIPPER PINCHER -->
+<!-- LEFT GRIPPER PINCHER -->
   <link name="l_gripper_pincher">
     <visual>
       <origin xyz="0 0 0" rpy="0 0 0" />
       <geometry>
-	<mesh filename="package://clam_description/stl/l_gripper_pincher.STL" scale="${M_SCALE}" />
+	<mesh filename="package://clam_description/stl/l_gripper_pincher.STL" scale="1 1 1" />
       </geometry>
       <material name="Black" />
     </visual>
-  </link>
-  <!-- RIGHT GRIPPER PINCHER -->
+    <collision>
+      <origin xyz="0 0 0" rpy="0 0 0" />
+      <geometry>
+	<mesh filename="package://clam_description/stl/l_gripper_pincher.STL" scale="1 1 1" />
+      </geometry>
+    </collision>
+  </link>
+<!-- RIGHT GRIPPER PINCHER -->
   <link name="r_gripper_pincher">
     <visual>
       <origin xyz="0 0 0" rpy="0 0 0" />
       <geometry>
-	<mesh filename="package://clam_description/stl/r_gripper_pincher.STL" scale="${M_SCALE}" />
+	<mesh filename="package://clam_description/stl/r_gripper_pincher.STL" scale="1 1 1" />
       </geometry>
       <material name="Black" />
     </visual>
+    <collision>
+      <origin xyz="0 0 0" rpy="0 0 0" />
+      <geometry>
+	<mesh filename="package://clam_description/stl/r_gripper_pincher.STL" scale="1 1 1" />
+      </geometry>
+    </collision>
   </link>
 </robot>
