Commit message: Bug fixes for clam_interactive_markers issues

File: clam_description/urdf/clam_urdf.xacro (robot description, xacro)
@@ -11,6 +11,12 @@
      http://www.ros.org/wiki/xacro
 -->
-<robot name="clam">
+<robot name="clam"
+    xmlns:sensor="http://playerstage.sourceforge.net/gazebo/xmlschema/#sensor"
+    xmlns:controller="http://playerstage.sourceforge.net/gazebo/xmlschema/#controller"
+    xmlns:interface="http://playerstage.sourceforge.net/gazebo/xmlschema/#interface">
+  <!-- Include materials -->
   <include filename="$(find clam_description)/urdf/materials.urdf.xacro" />
+  <!-- Constants -->
+  <property name="M_SCALE" value="0.001"/>
   <!-- BASE LINK -->
   <link name="base_link">
@@ -18,5 +24,5 @@
       <origin xyz="0 0 0" rpy="1.5708 0 0" /> <!-- rotate PI/2 -->
       <geometry>
-	<mesh filename="package://clam_description/cad/arm_assemblies/stl/base_link.STL" scale=".001 .001 .001" />
+	<mesh filename="package://clam_description/cad/arm_assemblies/stl/base_link.STL" scale="${M_SCALE} ${M_SCALE} ${M_SCALE}" />
 	<!--box size="0.1 0.1 0.05" /-->
       </geometry>
@@ -26,5 +32,5 @@
       <origin xyz="0 0 0" rpy="1.5708 0 0" />
       <geometry>
-	<mesh filename="package://clam_description/cad/arm_assemblies/stl/base_link_convex.STL" scale=".001 .001 .001" />
+	<mesh filename="package://clam_description/cad/arm_assemblies/stl/base_link_convex.STL" scale="${M_SCALE} ${M_SCALE} ${M_SCALE}" />
       </geometry>>
     </collision-->
@@ -47,5 +53,5 @@
       <origin xyz="0 0 0" rpy="1.5708 0 0" />
       <geometry>
-	<mesh filename="package://clam_description/cad/arm_assemblies/stl/shoulder_pan_link.STL" scale=".001 .001 .001" />
+	<mesh filename="package://clam_description/cad/arm_assemblies/stl/shoulder_pan_link.STL" scale="${M_SCALE} ${M_SCALE} ${M_SCALE}" />
 	<!--cylinder length="0.046" radius="0.03" /-->
       </geometry>
@@ -66,5 +72,5 @@
       <origin xyz="-0.002 0 -0.005" rpy="1.5708 3.1416 1.5708" />
       <geometry>
-	<mesh filename="package://clam_description/cad/arm_assemblies/stl/shoulder_pitch_link.STL" scale=".001 .001 .001" />
+	<mesh filename="package://clam_description/cad/arm_assemblies/stl/shoulder_pitch_link.STL" scale="${M_SCALE} ${M_SCALE} ${M_SCALE}" />
 	<!--cylinder length="0.117" radius="0.02" /-->
       </geometry>
@@ -74,5 +80,5 @@
       <origin xyz="-0.002 0 -0.005" rpy="1.5708 3.1416 1.5708" />
       <geometry>
-	<mesh filename="package://clam_description/cad/arm_assemblies/stl/shoulder_pitch_link_convex.STL" scale=".001 .001 .001" />
+	<mesh filename="package://clam_description/cad/arm_assemblies/stl/shoulder_pitch_link_convex.STL" scale="${M_SCALE} ${M_SCALE} ${M_SCALE}" />
       </geometry>
     </collision-->
@@ -91,5 +97,5 @@
       <origin xyz="-0.006 0.0 ${0.039 * 0}" rpy="1.5708 3.1416 0" />
       <geometry>
-	<mesh filename="package://clam_description/cad/arm_assemblies/stl/elbow_roll_link.STL" scale=".001 .001 .001" />
+	<mesh filename="package://clam_description/cad/arm_assemblies/stl/elbow_roll_link.STL" scale="${M_SCALE} ${M_SCALE} ${M_SCALE}" />
 	<!--cylinder length="0.039" radius="0.02" /-->
       </geometry>
@@ -110,5 +116,5 @@
       <origin xyz="-0.004 0 ${0.215 * 0}" rpy="1.5708 3.1416 4.7124" />
       <geometry>
-	<mesh filename="package://clam_description/cad/arm_assemblies/stl/elbow_pitch_link.STL" scale=".001 .001 .001" />
+	<mesh filename="package://clam_description/cad/arm_assemblies/stl/elbow_pitch_link.STL" scale="${M_SCALE} ${M_SCALE} ${M_SCALE}" />
 	<!--cylinder length="0.215" radius="0.02" /-->
       </geometry>
@@ -129,5 +135,5 @@
       <origin xyz="0 0 0" rpy="-1.5708 0 0" />
       <geometry>
-	<mesh filename="package://clam_description/cad/arm_assemblies/stl/wrist_roll_link.STL" scale=".001 .001 .001" />
+	<mesh filename="package://clam_description/cad/arm_assemblies/stl/wrist_roll_link.STL" scale="${M_SCALE} ${M_SCALE} ${M_SCALE}" />
 	<!--cylinder length="0.033" radius="0.02" /-->
       </geometry>
@@ -138,5 +144,5 @@
     <parent link="wrist_roll_link"/>
     <child link="wrist_pitch_link"/>
-    <origin xyz="-0.001 0.000 0" rpy="0 0 0" />
+    <origin xyz="-0${M_SCALE} 0.000 0" rpy="0 0 0" />
     <axis xyz="1 0 0" />
     <limit effort="300" velocity="1" lower="-1.5953400194" upper="1.98394848567" />
@@ -148,5 +154,5 @@
       <origin xyz="0 0 0" rpy="3.1416 -1.5708 0" />
       <geometry>
-	<mesh filename="package://clam_description/cad/arm_assemblies/stl/wrist_pitch_link.STL" scale=".001 .001 .001" />
+	<mesh filename="package://clam_description/cad/arm_assemblies/stl/wrist_pitch_link.STL" scale="${M_SCALE} ${M_SCALE} ${M_SCALE}" />
 	<!--cylinder length="0.081" radius="0.02" /-->
       </geometry>

Commit message: Moved location of stl files to root fo clam_description Updated urdf file to all have same axis of rotation for use with interactive_markers

File: clam_description/urdf/clam_urdf.xacro (robot description, xacro)
@@ -19,10 +19,11 @@
   <!-- Constants -->
   <property name="M_SCALE" value="0.001"/>
+  <property name="M_PI" value="3.14159"/>
   <!-- BASE LINK -->
   <link name="base_link">
     <visual>
-      <origin xyz="0 0 0" rpy="1.5708 0 0" /> <!-- rotate PI/2 -->
+      <origin xyz="0 0 0" rpy="${M_PI/2} 0 0" /> <!-- rotate PI/2 -->
       <geometry>
-	<mesh filename="package://clam_description/cad/arm_assemblies/stl/base_link.STL" scale="${M_SCALE} ${M_SCALE} ${M_SCALE}" />
+	<mesh filename="package://clam_description/stl/base_link.STL" scale="${M_SCALE} ${M_SCALE} ${M_SCALE}" />
 	<!--box size="0.1 0.1 0.05" /-->
       </geometry>
@@ -30,7 +31,7 @@
     </visual>
     <!--collision>
-      <origin xyz="0 0 0" rpy="1.5708 0 0" />
+      <origin xyz="0 0 0" rpy="${M_PI/2} 0 0" />
       <geometry>
-	<mesh filename="package://clam_description/cad/arm_assemblies/stl/base_link_convex.STL" scale="${M_SCALE} ${M_SCALE} ${M_SCALE}" />
+	<mesh filename="package://clam_description/stl/base_link_convex.STL" scale="${M_SCALE} ${M_SCALE} ${M_SCALE}" />
       </geometry>>
     </collision-->
@@ -43,6 +44,6 @@
     <parent link="base_link"/>
     <child link="shoulder_pan_link"/>
-    <origin xyz="0 0 0.05" rpy="0 0 0" />
-    <axis xyz="0 0 1" />
+    <origin xyz="0 0 0.05" rpy="0 ${M_PI/2} 0" />
+    <axis xyz="1 0 0" />
     <limit effort="300" velocity="1" lower="-2.61799387799" upper="1.98394848567"/>
     <dynamics damping="50" friction="1"/>
@@ -51,7 +52,7 @@
   <link name="shoulder_pan_link" >
     <visual>
-      <origin xyz="0 0 0" rpy="1.5708 0 0" />
+      <origin xyz="0 0 0" rpy="0 0 ${M_PI/2}" />
       <geometry>
-	<mesh filename="package://clam_description/cad/arm_assemblies/stl/shoulder_pan_link.STL" scale="${M_SCALE} ${M_SCALE} ${M_SCALE}" />
+	<mesh filename="package://clam_description/stl/shoulder_pan_link.STL" scale="${M_SCALE} ${M_SCALE} ${M_SCALE}" />
 	<!--cylinder length="0.046" radius="0.03" /-->
       </geometry>
@@ -62,5 +63,5 @@
     <parent link="shoulder_pan_link"/>
     <child link="shoulder_pitch_link"/>
-    <origin xyz="0 0.0 ${0.046 * 1}" rpy="0 0 0" />
+    <origin xyz="0 0 ${0.046 * 0}" rpy="-${M_PI/2} 0 ${M_PI/2}" />
     <axis xyz="1 0 0" />
     <limit effort="300" velocity="1" lower="-1.19962513147" upper="1.89994105047" />
@@ -70,7 +71,7 @@
   <link name="shoulder_pitch_link" >
     <visual>
-      <origin xyz="-0.002 0 -0.005" rpy="1.5708 3.1416 1.5708" />
+      <origin xyz="-0.002 0 0.046" rpy="${M_PI/2} ${M_PI} ${M_PI/2}" />
       <geometry>
-	<mesh filename="package://clam_description/cad/arm_assemblies/stl/shoulder_pitch_link.STL" scale="${M_SCALE} ${M_SCALE} ${M_SCALE}" />
+	<mesh filename="package://clam_description/stl/shoulder_pitch_link.STL" scale="${M_SCALE} ${M_SCALE} ${M_SCALE}" />
 	<!--cylinder length="0.117" radius="0.02" /-->
       </geometry>
@@ -78,7 +79,7 @@
     </visual>
     <!--collision>
-      <origin xyz="-0.002 0 -0.005" rpy="1.5708 3.1416 1.5708" />
+      <origin xyz="-0.002 0 -0.005" rpy="${M_PI/2} ${M_PI} ${M_PI/2}" />
       <geometry>
-	<mesh filename="package://clam_description/cad/arm_assemblies/stl/shoulder_pitch_link_convex.STL" scale="${M_SCALE} ${M_SCALE} ${M_SCALE}" />
+	<mesh filename="package://clam_description/stl/shoulder_pitch_link_convex.STL" scale="${M_SCALE} ${M_SCALE} ${M_SCALE}" />
       </geometry>
     </collision-->
@@ -88,5 +89,5 @@
     <child link="elbow_roll_link"/>
     <origin xyz="0.004 0 ${0.117 * 1 + 0.035}" rpy="0 0 0" />
-    <axis xyz="0 0 1" />
+    <axis xyz="1 0 0" />
     <limit effort="300" velocity="1" lower="-2.61799387799" upper="0.705631162427" />
     <dynamics damping="50" friction="1"/>
@@ -95,7 +96,7 @@
   <link name="elbow_roll_link" >
     <visual>
-      <origin xyz="-0.006 0.0 ${0.039 * 0}" rpy="1.5708 3.1416 0" />
+      <origin xyz="-0.006 0.0 ${0.039 * 0}" rpy="${M_PI/2} ${M_PI} 0" />
       <geometry>
-	<mesh filename="package://clam_description/cad/arm_assemblies/stl/elbow_roll_link.STL" scale="${M_SCALE} ${M_SCALE} ${M_SCALE}" />
+	<mesh filename="package://clam_description/stl/elbow_roll_link.STL" scale="${M_SCALE} ${M_SCALE} ${M_SCALE}" />
 	<!--cylinder length="0.039" radius="0.02" /-->
       </geometry>
@@ -114,7 +115,7 @@
   <link name="elbow_pitch_link" >
     <visual>
-      <origin xyz="-0.004 0 ${0.215 * 0}" rpy="1.5708 3.1416 4.7124" />
+      <origin xyz="-0.004 0 ${0.215 * 0}" rpy="${M_PI/2} ${M_PI} 4.7124" />
       <geometry>
-	<mesh filename="package://clam_description/cad/arm_assemblies/stl/elbow_pitch_link.STL" scale="${M_SCALE} ${M_SCALE} ${M_SCALE}" />
+	<mesh filename="package://clam_description/stl/elbow_pitch_link.STL" scale="${M_SCALE} ${M_SCALE} ${M_SCALE}" />
 	<!--cylinder length="0.215" radius="0.02" /-->
       </geometry>
@@ -126,5 +127,5 @@
     <child link="wrist_roll_link"/>
     <origin xyz="-0.004 -0.008 ${0.215 * 1 + 0.033}" rpy="0 0 0" />
-    <axis xyz="0 0 1" />
+    <axis xyz="1 0 0" />
     <limit effort="300" velocity="1" lower="-2.61799387799" upper="2.6128806087" />
     <dynamics damping="50" friction="1"/>
@@ -133,7 +134,7 @@
   <link name="wrist_roll_link" >
     <visual>
-      <origin xyz="0 0 0" rpy="-1.5708 0 0" />
+      <origin xyz="0 0 0" rpy="-${M_PI/2} 0 0" />
       <geometry>
-	<mesh filename="package://clam_description/cad/arm_assemblies/stl/wrist_roll_link.STL" scale="${M_SCALE} ${M_SCALE} ${M_SCALE}" />
+	<mesh filename="package://clam_description/stl/wrist_roll_link.STL" scale="${M_SCALE} ${M_SCALE} ${M_SCALE}" />
 	<!--cylinder length="0.033" radius="0.02" /-->
       </geometry>
@@ -152,7 +153,7 @@
   <link name="wrist_pitch_link">
     <visual>
-      <origin xyz="0 0 0" rpy="3.1416 -1.5708 0" />
+      <origin xyz="0 0 0" rpy="${M_PI} -${M_PI/2} 0" />
       <geometry>
-	<mesh filename="package://clam_description/cad/arm_assemblies/stl/wrist_pitch_link.STL" scale="${M_SCALE} ${M_SCALE} ${M_SCALE}" />
+	<mesh filename="package://clam_description/stl/wrist_pitch_link.STL" scale="${M_SCALE} ${M_SCALE} ${M_SCALE}" />
 	<!--cylinder length="0.081" radius="0.02" /-->
       </geometry>
@@ -164,5 +165,5 @@
     <child link="gripper_roll_link"/>
     <origin xyz="0 0 ${0.081 * 1}" rpy="0 0 0" />
-    <axis xyz="0 0 1" />
+    <axis xyz="1 0 0" />
     <limit effort="300" velocity="1" lower="-2.61799387799" upper="2.6128806087" />
     <dynamics damping="50" friction="1"/>

Commit message: Finished converting first 3 joints of arm to same axis movement

File: clam_description/urdf/clam_urdf.xacro (robot description, xacro)
@@ -63,5 +63,5 @@
     <parent link="shoulder_pan_link"/>
     <child link="shoulder_pitch_link"/>
-    <origin xyz="0 0 ${0.046 * 0}" rpy="-${M_PI/2} 0 ${M_PI/2}" />
+    <origin xyz="-0.041 0.0 0.0" rpy="-${M_PI/2} 0 ${M_PI/2}" />
     <axis xyz="1 0 0" />
     <limit effort="300" velocity="1" lower="-1.19962513147" upper="1.89994105047" />
@@ -71,5 +71,5 @@
   <link name="shoulder_pitch_link" >
     <visual>
-      <origin xyz="-0.002 0 0.046" rpy="${M_PI/2} ${M_PI} ${M_PI/2}" />
+      <origin xyz="-0.002 0 -0.000" rpy="${M_PI/2} ${M_PI} ${M_PI/2}" />
       <geometry>
 	<mesh filename="package://clam_description/stl/shoulder_pitch_link.STL" scale="${M_SCALE} ${M_SCALE} ${M_SCALE}" />
@@ -78,15 +78,9 @@
       <material name="Grey" />
     </visual>
-    <!--collision>
-      <origin xyz="-0.002 0 -0.005" rpy="${M_PI/2} ${M_PI} ${M_PI/2}" />
-      <geometry>
-	<mesh filename="package://clam_description/stl/shoulder_pitch_link_convex.STL" scale="${M_SCALE} ${M_SCALE} ${M_SCALE}" />
-      </geometry>
-    </collision-->
   </link>
   <joint name="elbow_roll_joint" type="revolute">
     <parent link="shoulder_pitch_link"/>
     <child link="elbow_roll_link"/>
-    <origin xyz="0.004 0 ${0.117 * 1 + 0.035}" rpy="0 0 0" />
+    <origin xyz="-0.001 0 0.121" rpy="0 ${M_PI/2} 0" />
     <axis xyz="1 0 0" />
     <limit effort="300" velocity="1" lower="-2.61799387799" upper="0.705631162427" />
@@ -94,7 +88,8 @@
   </joint>
   <!-- ELBOW ROLL LINK -->
+  <!-- CONTINUE CONVERTING URDF HERE -->
   <link name="elbow_roll_link" >
     <visual>
-      <origin xyz="-0.006 0.0 ${0.039 * 0}" rpy="${M_PI/2} ${M_PI} 0" />
+      <origin xyz="0.0 0.0 0.0" rpy="${M_PI} ${M_PI/2} ${M_PI/2}" />
       <geometry>
 	<mesh filename="package://clam_description/stl/elbow_roll_link.STL" scale="${M_SCALE} ${M_SCALE} ${M_SCALE}" />

Commit message: Finished re-making the URDF file Fixed the marker server to work with joints correctly

File: clam_description/urdf/clam_urdf.xacro (robot description, xacro)
@@ -44,6 +44,6 @@
     <parent link="base_link"/>
     <child link="shoulder_pan_link"/>
-    <origin xyz="0 0 0.05" rpy="0 ${M_PI/2} 0" />
-    <axis xyz="1 0 0" />
+    <origin xyz="0 0 0.05" rpy="0 ${M_PI/2} ${M_PI*0}" />
+    <axis xyz="-1 0 0" />
     <limit effort="300" velocity="1" lower="-2.61799387799" upper="1.98394848567"/>
     <dynamics damping="50" friction="1"/>
@@ -82,14 +82,13 @@
     <parent link="shoulder_pitch_link"/>
     <child link="elbow_roll_link"/>
-    <origin xyz="-0.001 0 0.121" rpy="0 ${M_PI/2} 0" />
-    <axis xyz="1 0 0" />
+    <origin xyz="-0.001 0 0.121" rpy="${M_PI} ${M_PI/2} 0" />
+    <axis xyz="-1 0 0" />
     <limit effort="300" velocity="1" lower="-2.61799387799" upper="0.705631162427" />
     <dynamics damping="50" friction="1"/>
   </joint>
   <!-- ELBOW ROLL LINK -->
-  <!-- CONTINUE CONVERTING URDF HERE -->
   <link name="elbow_roll_link" >
     <visual>
-      <origin xyz="0.0 0.0 0.0" rpy="${M_PI} ${M_PI/2} ${M_PI/2}" />
+      <origin xyz="-0.035 0.0 0.0" rpy="${M_PI} ${M_PI/2} ${M_PI/2}" />
       <geometry>
 	<mesh filename="package://clam_description/stl/elbow_roll_link.STL" scale="${M_SCALE} ${M_SCALE} ${M_SCALE}" />
@@ -102,5 +101,5 @@
     <parent link="elbow_roll_link"/>
     <child link="elbow_pitch_link"/>
-    <origin xyz="0 0 ${0.215 * 0}" rpy="0 0 0" />
+    <origin xyz="-0.035 0 0.0009" rpy="0 ${M_PI/2} 0" />
     <axis xyz="1 0 0" />
     <limit effort="300" velocity="1" lower="-1.5953400194" upper="1.93281579274" />
@@ -110,5 +109,6 @@
   <link name="elbow_pitch_link" >
     <visual>
-      <origin xyz="-0.004 0 ${0.215 * 0}" rpy="${M_PI/2} ${M_PI} 4.7124" />
+      <!--   roll   pitch=green  yaw=blue axis -->
+      <origin xyz="0.0 0 -${0.035*0}" rpy="${M_PI/2} 0 ${M_PI/2+M_PI}" />
       <geometry>
 	<mesh filename="package://clam_description/stl/elbow_pitch_link.STL" scale="${M_SCALE} ${M_SCALE} ${M_SCALE}" />
@@ -121,5 +121,5 @@
     <parent link="elbow_pitch_link"/>
     <child link="wrist_roll_link"/>
-    <origin xyz="-0.004 -0.008 ${0.215 * 1 + 0.033}" rpy="0 0 0" />
+    <origin xyz="0.0 -0.008 -.248" rpy="0 ${M_PI/2} ${M_PI}" />
     <axis xyz="1 0 0" />
     <limit effort="300" velocity="1" lower="-2.61799387799" upper="2.6128806087" />
@@ -129,5 +129,5 @@
   <link name="wrist_roll_link" >
     <visual>
-      <origin xyz="0 0 0" rpy="-${M_PI/2} 0 0" />
+      <origin xyz="0 0 0" rpy="0 ${M_PI/2} ${M_PI/2}" />
       <geometry>
 	<mesh filename="package://clam_description/stl/wrist_roll_link.STL" scale="${M_SCALE} ${M_SCALE} ${M_SCALE}" />
@@ -140,5 +140,5 @@
     <parent link="wrist_roll_link"/>
     <child link="wrist_pitch_link"/>
-    <origin xyz="-0${M_SCALE} 0.000 0" rpy="0 0 0" />
+    <origin xyz="0.0 0.0 0.002" rpy="0 ${M_PI/2} 0" />
     <axis xyz="1 0 0" />
     <limit effort="300" velocity="1" lower="-1.5953400194" upper="1.98394848567" />
@@ -159,5 +159,5 @@
     <parent link="wrist_pitch_link"/>
     <child link="gripper_roll_link"/>
-    <origin xyz="0 0 ${0.081 * 1}" rpy="0 0 0" />
+    <origin xyz="0 0 0.1" rpy="0 ${M_PI/2} 0" />
     <axis xyz="1 0 0" />
     <limit effort="300" velocity="1" lower="-2.61799387799" upper="2.6128806087" />
@@ -167,7 +167,7 @@
   <link name="gripper_roll_link">
     <visual>
-      <origin xyz="0 0 ${0.040 * .5}" rpy="0 0 0" />
+      <origin xyz="0 0 0" rpy="0 ${M_PI/2} 0" />
       <geometry>
-	<cylinder length="0.040" radius="0.025" />
+	<box size="0.06 0.015 0.04" />
       </geometry>
       <material name="Orange" />
@@ -177,5 +177,5 @@
     <parent link="gripper_roll_link"/>
     <child link="gripper_grip_link"/>
-    <origin xyz="0 0 ${0.040 * 1}" rpy="0 0 0" />
+    <origin xyz="-0.02 0 0.0" rpy="0 0 ${M_PI/2}" />
     <axis xyz="1 0 0" />
     <limit effort="300" velocity="1" lower="-0.940841549903" upper="0.0" />
@@ -185,7 +185,7 @@
   <link name="gripper_grip_link">
     <visual>
-      <origin xyz="0 0 ${0.060 * .5}" rpy="0 0 0" />
+      <origin xyz="0.0 0.03 0" rpy="${M_PI/2} 0 0" />
       <geometry>
-	<box size="0.03 0.02 0.060" />
+	<box size="0.03 0.005 0.060" />
       </geometry>
       <material name="Black" />

Commit message: Modified URDF files to have collision models. Still broken.

File: clam_description/urdf/clam_urdf.xacro (robot description, xacro)
@@ -30,10 +30,10 @@
       <material name="Grey" />
     </visual>
-    <!--collision>
-      <origin xyz="0 0 0" rpy="${M_PI/2} 0 0" />
-      <geometry>
-	<mesh filename="package://clam_description/stl/base_link_convex.STL" scale="${M_SCALE} ${M_SCALE} ${M_SCALE}" />
-      </geometry>>
-    </collision-->
+    <collision>
+      <origin xyz="0 0 0" rpy="${M_PI/2} 0 0" /> <!-- rotate PI/2 -->
+      <geometry>
+	<mesh filename="package://clam_description/stl/base_link_simple.STL" scale="${M_SCALE} ${M_SCALE} ${M_SCALE}" />
+      </geometry>
+    </collision>>
     <inertial>
       <mass value="25" />
@@ -55,8 +55,13 @@
       <geometry>
 	<mesh filename="package://clam_description/stl/shoulder_pan_link.STL" scale="${M_SCALE} ${M_SCALE} ${M_SCALE}" />
-	<!--cylinder length="0.046" radius="0.03" /-->
       </geometry>
       <material name="Orange" />
     </visual>
+    <collision>
+      <origin xyz="0 0 0" rpy="0 0 ${M_PI/2}" />
+      <geometry>
+	<mesh filename="package://clam_description/stl/shoulder_pan_link_simple.STL" scale="${M_SCALE} ${M_SCALE} ${M_SCALE}" />
+      </geometry>
+    </collision>
   </link>
   <joint name="shoulder_pitch_joint" type="revolute">
@@ -74,8 +79,13 @@
       <geometry>
 	<mesh filename="package://clam_description/stl/shoulder_pitch_link.STL" scale="${M_SCALE} ${M_SCALE} ${M_SCALE}" />
-	<!--cylinder length="0.117" radius="0.02" /-->
       </geometry>
       <material name="Grey" />
     </visual>
+    <collision>
+      <origin xyz="-0.002 0 -0.000" rpy="${M_PI/2} ${M_PI} ${M_PI/2}" />
+      <geometry>
+	<mesh filename="package://clam_description/stl/shoulder_pitch_link_simple.STL" scale="${M_SCALE} ${M_SCALE} ${M_SCALE}" />
+      </geometry>
+    </collision>
   </link>
   <joint name="elbow_roll_joint" type="revolute">
@@ -93,8 +103,13 @@
       <geometry>
 	<mesh filename="package://clam_description/stl/elbow_roll_link.STL" scale="${M_SCALE} ${M_SCALE} ${M_SCALE}" />
-	<!--cylinder length="0.039" radius="0.02" /-->
       </geometry>
       <material name="Black" />
     </visual>
+    <collision>
+      <origin xyz="-0.035 0.0 0.0" rpy="${M_PI} ${M_PI/2} ${M_PI/2}" />
+      <geometry>
+	<mesh filename="package://clam_description/stl/elbow_roll_link_simple.STL" scale="${M_SCALE} ${M_SCALE} ${M_SCALE}" />
+      </geometry>
+    </collision>
   </link>
   <joint name="elbow_pitch_joint" type="revolute">
@@ -109,12 +124,16 @@
   <link name="elbow_pitch_link" >
     <visual>
-      <!--   roll   pitch=green  yaw=blue axis -->
       <origin xyz="0.0 0 -${0.035*0}" rpy="${M_PI/2} 0 ${M_PI/2+M_PI}" />
       <geometry>
 	<mesh filename="package://clam_description/stl/elbow_pitch_link.STL" scale="${M_SCALE} ${M_SCALE} ${M_SCALE}" />
-	<!--cylinder length="0.215" radius="0.02" /-->
       </geometry>
       <material name="Orange" />
     </visual>
+    <collision>
+      <origin xyz="0.0 0 -${0.035*0}" rpy="${M_PI/2} 0 ${M_PI/2+M_PI}" />
+      <geometry>
+	<mesh filename="package://clam_description/stl/elbow_pitch_link_simple.STL" scale="${M_SCALE} ${M_SCALE} ${M_SCALE}" />
+      </geometry>
+    </collision>
   </link>
   <joint name="wrist_roll_joint" type="revolute">
@@ -136,4 +155,11 @@
       <material name="Black" />
     </visual>
+    <collision>
+      <origin xyz="0 0 0" rpy="0 ${M_PI/2} ${M_PI/2}" />
+      <geometry>
+	<mesh filename="package://clam_description/stl/wrist_roll_link_simple.STL" scale="${M_SCALE} ${M_SCALE} ${M_SCALE}" />
+	<!--cylinder length="0.033" radius="0.02" /-->
+      </geometry>
+    </collision>
   </link>
   <joint name="wrist_pitch_joint" type="revolute">
@@ -151,8 +177,13 @@
       <geometry>
 	<mesh filename="package://clam_description/stl/wrist_pitch_link.STL" scale="${M_SCALE} ${M_SCALE} ${M_SCALE}" />
-	<!--cylinder length="0.081" radius="0.02" /-->
       </geometry>
       <material name="Grey" />
     </visual>
+    <collision>
+      <origin xyz="0 0 0" rpy="${M_PI} -${M_PI/2} 0" />
+      <geometry>
+	<mesh filename="package://clam_description/stl/wrist_pitch_link_simple.STL" scale="${M_SCALE} ${M_SCALE} ${M_SCALE}" />
+      </geometry>
+    </collision>
   </link>
   <joint name="gripper_roll_joint" type="revolute">
