Commit message: Simplified urdf scale code

File: clam_description/urdf/clam_urdf.xacro (robot description, xacro)
@@ -18,5 +18,5 @@
   <include filename="$(find clam_description)/urdf/materials.urdf.xacro" />
   <!-- Constants -->
-  <property name="M_SCALE" value="0.001"/>
+  <property name="M_SCALE" value="0.001 0.001 0.001"/>
   <property name="M_PI" value="3.14159"/>
   <!-- BASE LINK -->
@@ -25,6 +25,5 @@
       <origin xyz="0 0 0" rpy="${M_PI/2} 0 0" /> <!-- rotate PI/2 -->
       <geometry>
-	<mesh filename="package://clam_description/stl/base_link.STL" scale="${M_SCALE} ${M_SCALE} ${M_SCALE}" />
-	<!--box size="0.1 0.1 0.05" /-->
+	<mesh filename="package://clam_description/stl/base_link.STL" scale="${M_SCALE}" />
       </geometry>
       <material name="Grey" />
@@ -33,5 +32,5 @@
       <origin xyz="0 0 0" rpy="${M_PI/2} 0 0" /> <!-- rotate PI/2 -->
       <geometry>
-	<mesh filename="package://clam_description/stl/base_link_simple.STL" scale="${M_SCALE} ${M_SCALE} ${M_SCALE}" />
+	<mesh filename="package://clam_description/stl/base_link_simple.STL" scale="${M_SCALE}" />
       </geometry>
     </collision>>
@@ -54,5 +53,5 @@
       <origin xyz="0 0 0" rpy="0 0 ${M_PI/2}" />
       <geometry>
-	<mesh filename="package://clam_description/stl/shoulder_pan_link.STL" scale="${M_SCALE} ${M_SCALE} ${M_SCALE}" />
+	<mesh filename="package://clam_description/stl/shoulder_pan_link.STL" scale="${M_SCALE}" />
       </geometry>
       <material name="Orange" />
@@ -61,5 +60,5 @@
       <origin xyz="0 0 0" rpy="0 0 ${M_PI/2}" />
       <geometry>
-	<mesh filename="package://clam_description/stl/shoulder_pan_link_simple.STL" scale="${M_SCALE} ${M_SCALE} ${M_SCALE}" />
+	<mesh filename="package://clam_description/stl/shoulder_pan_link_simple.STL" scale="${M_SCALE}" />
       </geometry>
     </collision>
@@ -78,5 +77,5 @@
       <origin xyz="-0.002 0 -0.000" rpy="${M_PI/2} ${M_PI} ${M_PI/2}" />
       <geometry>
-	<mesh filename="package://clam_description/stl/shoulder_pitch_link.STL" scale="${M_SCALE} ${M_SCALE} ${M_SCALE}" />
+	<mesh filename="package://clam_description/stl/shoulder_pitch_link.STL" scale="${M_SCALE}" />
       </geometry>
       <material name="Grey" />
@@ -85,5 +84,5 @@
       <origin xyz="-0.002 0 -0.000" rpy="${M_PI/2} ${M_PI} ${M_PI/2}" />
       <geometry>
-	<mesh filename="package://clam_description/stl/shoulder_pitch_link_simple.STL" scale="${M_SCALE} ${M_SCALE} ${M_SCALE}" />
+	<mesh filename="package://clam_description/stl/shoulder_pitch_link_simple.STL" scale="${M_SCALE}" />
       </geometry>
     </collision>
@@ -102,5 +101,5 @@
       <origin xyz="-0.035 0.0 0.0" rpy="${M_PI} ${M_PI/2} ${M_PI/2}" />
       <geometry>
-	<mesh filename="package://clam_description/stl/elbow_roll_link.STL" scale="${M_SCALE} ${M_SCALE} ${M_SCALE}" />
+	<mesh filename="package://clam_description/stl/elbow_roll_link.STL" scale="${M_SCALE}" />
       </geometry>
       <material name="Black" />
@@ -109,5 +108,5 @@
       <origin xyz="-0.035 0.0 0.0" rpy="${M_PI} ${M_PI/2} ${M_PI/2}" />
       <geometry>
-	<mesh filename="package://clam_description/stl/elbow_roll_link_simple.STL" scale="${M_SCALE} ${M_SCALE} ${M_SCALE}" />
+	<mesh filename="package://clam_description/stl/elbow_roll_link_simple.STL" scale="${M_SCALE}" />
       </geometry>
     </collision>
@@ -126,5 +125,5 @@
       <origin xyz="0.0 0 -${0.035*0}" rpy="${M_PI/2} 0 ${M_PI/2+M_PI}" />
       <geometry>
-	<mesh filename="package://clam_description/stl/elbow_pitch_link.STL" scale="${M_SCALE} ${M_SCALE} ${M_SCALE}" />
+	<mesh filename="package://clam_description/stl/elbow_pitch_link.STL" scale="${M_SCALE}" />
       </geometry>
       <material name="Orange" />
@@ -133,5 +132,5 @@
       <origin xyz="0.0 0 -${0.035*0}" rpy="${M_PI/2} 0 ${M_PI/2+M_PI}" />
       <geometry>
-	<mesh filename="package://clam_description/stl/elbow_pitch_link_simple.STL" scale="${M_SCALE} ${M_SCALE} ${M_SCALE}" />
+	<mesh filename="package://clam_description/stl/elbow_pitch_link_simple.STL" scale="${M_SCALE}" />
       </geometry>
     </collision>
@@ -150,5 +149,5 @@
       <origin xyz="0 0 0" rpy="0 ${M_PI/2} ${M_PI/2}" />
       <geometry>
-	<mesh filename="package://clam_description/stl/wrist_roll_link.STL" scale="${M_SCALE} ${M_SCALE} ${M_SCALE}" />
+	<mesh filename="package://clam_description/stl/wrist_roll_link.STL" scale="${M_SCALE}" />
 	<!--cylinder length="0.033" radius="0.02" /-->
       </geometry>
@@ -158,5 +157,5 @@
       <origin xyz="0 0 0" rpy="0 ${M_PI/2} ${M_PI/2}" />
       <geometry>
-	<mesh filename="package://clam_description/stl/wrist_roll_link_simple.STL" scale="${M_SCALE} ${M_SCALE} ${M_SCALE}" />
+	<mesh filename="package://clam_description/stl/wrist_roll_link_simple.STL" scale="${M_SCALE}" />
 	<!--cylinder length="0.033" radius="0.02" /-->
       </geometry>
@@ -176,5 +175,5 @@
       <origin xyz="0 0 0" rpy="${M_PI} -${M_PI/2} 0" />
       <geometry>
-	<mesh filename="package://clam_description/stl/wrist_pitch_link.STL" scale="${M_SCALE} ${M_SCALE} ${M_SCALE}" />
+	<mesh filename="package://clam_description/stl/wrist_pitch_link.STL" scale="${M_SCALE}" />
       </geometry>
       <material name="Grey" />
@@ -183,5 +182,5 @@
       <origin xyz="0 0 0" rpy="${M_PI} -${M_PI/2} 0" />
       <geometry>
-	<mesh filename="package://clam_description/stl/wrist_pitch_link_simple.STL" scale="${M_SCALE} ${M_SCALE} ${M_SCALE}" />
+	<mesh filename="package://clam_description/stl/wrist_pitch_link_simple.STL" scale="${M_SCALE}" />
       </geometry>
     </collision>
@@ -218,5 +217,5 @@
       <origin xyz="0.0 0.03 0" rpy="${M_PI/2} 0 0" />
       <geometry>
-	<!--mesh filename="package://clam_description/stl/gripper.dae" scale="${M_SCALE} ${M_SCALE} ${M_SCALE}" /-->
+	<!--mesh filename="package://clam_description/stl/gripper.dae" scale="${M_SCALE}" /-->
 	<box size="0.03 0.005 0.060" />
       </geometry>

Commit message: Updated URDF file with collision model

File: clam_description/urdf/clam_urdf.xacro (robot description, xacro)
@@ -139,5 +139,5 @@
     <parent link="elbow_pitch_link"/>
     <child link="wrist_roll_link"/>
-    <origin xyz="0.0 -0.008 -.248" rpy="0 ${M_PI/2} ${M_PI}" />
+    <origin xyz="0.0 0.008 -.248" rpy="0 ${M_PI/2} ${M_PI}" />
     <axis xyz="1 0 0" />
     <limit effort="300" velocity="1" lower="-2.61799387799" upper="2.6128806087" />
@@ -150,5 +150,4 @@
       <geometry>
 	<mesh filename="package://clam_description/stl/wrist_roll_link.STL" scale="${M_SCALE}" />
-	<!--cylinder length="0.033" radius="0.02" /-->
       </geometry>
       <material name="Black" />
@@ -158,5 +157,4 @@
       <geometry>
 	<mesh filename="package://clam_description/stl/wrist_roll_link_simple.STL" scale="${M_SCALE}" />
-	<!--cylinder length="0.033" radius="0.02" /-->
       </geometry>
     </collision>
@@ -165,5 +163,5 @@
     <parent link="wrist_roll_link"/>
     <child link="wrist_pitch_link"/>
-    <origin xyz="0.0 0.0 0.002" rpy="0 ${M_PI/2} 0" />
+    <origin xyz="0.0 0.0 ${1*0.002}" rpy="0 ${M_PI/2} 0" />
     <axis xyz="1 0 0" />
     <limit effort="300" velocity="1" lower="-1.5953400194" upper="1.98394848567" />

Commit message: Added gripper model, new arm_navigation package and attempted to mimick joints

File: clam_description/urdf/clam_urdf.xacro (robot description, xacro)
@@ -195,5 +195,5 @@
   <link name="gripper_roll_link">
     <visual>
-      <origin xyz="0 0 0" rpy="0 0 0" />
+      <origin xyz="0 .045 0" rpy="0 0 0" />
       <geometry>
 	<mesh filename="package://clam_description/stl/gripper_grip_link.STL" scale="${M_SCALE}" />
@@ -205,5 +205,5 @@
     <parent link="gripper_roll_link"/>
     <child link="l_gripper_aft_link"/>
-    <origin xyz="0.025 -0.0275 0" rpy="0 -${M_PI/2} ${34.58*M_PI/180}" />
+    <origin xyz="0.025 ${-0.0275+.040} 0" rpy="0 -${M_PI/2} ${34.58*M_PI/180}" />
     <axis xyz="1 0 0" />
     <limit effort="300" velocity="1" lower="${0*M_PI/180}" upper="${53*M_PI/180}" />
@@ -213,5 +213,5 @@
     <parent link="gripper_roll_link"/>
     <child link="r_gripper_aft_link"/>
-    <origin xyz="0.025 -0.0561 0" rpy="0 -${M_PI/2} ${-34.58*M_PI/180}" />
+    <origin xyz="0.025 ${-0.0561+.040}  0" rpy="0 -${M_PI/2} ${-34.58*M_PI/180}" />
     <axis xyz="1 0 0" />
     <limit effort="300" velocity="1" lower="-3.14" upper="3.14" />
@@ -222,5 +222,5 @@
     <parent link="gripper_roll_link"/>
     <child link="l_gripper_fwd_link"/>
-    <origin xyz="0.05 -0.037 0.007" rpy="0 -${M_PI/2} ${214.58*M_PI/180}" />
+    <origin xyz="0.05 ${-0.037+.040} 0.007" rpy="0 -${M_PI/2} ${214.58*M_PI/180}" />
     <axis xyz="1 0 0" />
     <limit effort="300" velocity="1" lower="0" upper="1.57" />
@@ -231,5 +231,5 @@
     <parent link="gripper_roll_link"/>
     <child link="r_gripper_fwd_link"/>
-    <origin xyz="0.05 -0.047 0.007" rpy="0 -${M_PI/2} ${145.42*M_PI/180}" />
+    <origin xyz="0.05 ${-0.047+.040} 0.007" rpy="0 -${M_PI/2} ${145.42*M_PI/180}" />
     <axis xyz="1 0 0" />
     <limit effort="300" velocity="1" lower="-1.57" upper="0" />

Commit message: Merged Andy's updated STL files

File: clam_description/urdf/clam_urdf.xacro (robot description, xacro)
@@ -242,5 +242,5 @@
       <origin xyz="0 0 0" rpy="0 0 0" />
       <geometry>
-	<mesh filename="package://clam_description/stl/l_gripper_fwd_link.STL" scale="${M_SCALE}" />
+	<mesh filename="package://clam_description/stl/l_gripper_fwd_link.STL" scale="1 1 1" />
       </geometry>
       <material name="Grey" />
@@ -252,5 +252,5 @@
       <origin xyz="0 0 0" rpy="0 0 0" />
       <geometry>
-	<mesh filename="package://clam_description/stl/r_gripper_fwd_link.STL" scale="${M_SCALE}" />
+	<mesh filename="package://clam_description/stl/r_gripper_fwd_link.STL" scale="1 1 1" />
       </geometry>
       <material name="Grey" />
@@ -262,5 +262,5 @@
       <origin xyz="0 0 0" rpy="0 0 0" />
       <geometry>
-	<mesh filename="package://clam_description/stl/l_gripper_aft_link.STL" scale="${M_SCALE}" />
+	<mesh filename="package://clam_description/stl/l_gripper_aft_link.STL" scale="1 1 1" />
       </geometry>
       <material name="Grey" />
@@ -281,5 +281,5 @@
       <origin xyz="0 0 0" rpy="0 0 0" />
       <geometry>
-	<mesh filename="package://clam_description/stl/r_gripper_aft_link.STL" scale="${M_SCALE}" />
+	<mesh filename="package://clam_description/stl/r_gripper_aft_link.STL" scale="1 1 1" />
       </geometry>
       <material name="Grey" />
@@ -300,5 +300,5 @@
       <origin xyz="0 0 0" rpy="0 0 0" />
       <geometry>
-	<mesh filename="package://clam_description/stl/l_gripper_pincher.STL" scale="${M_SCALE}" />
+	<mesh filename="package://clam_description/stl/l_gripper_pincher.STL" scale="1 1 1" />
       </geometry>
       <material name="Black" />
@@ -310,5 +310,5 @@
       <origin xyz="0 0 0" rpy="0 0 0" />
       <geometry>
-	<mesh filename="package://clam_description/stl/r_gripper_pincher.STL" scale="${M_SCALE}" />
+	<mesh filename="package://clam_description/stl/r_gripper_pincher.STL" scale="1 1 1" />
       </geometry>
       <material name="Black" />

Commit message: Updated URDF to include kinect calibration and camera links

File: clam_description/urdf/clam_urdf.xacro (robot description, xacro)
@@ -315,3 +315,31 @@
     </visual>
   </link>
+  <!-- FAKE CAMERA CALIBRATION POINT -->
+  <joint name="gripper_link_joint" type="fixed">
+    <origin xyz="0.012 -0.11 0.020" rpy="0 0 0" />
+    <parent link="l_gripper_pincher"/>
+    <child link="gripper_link" />
+  </joint>
+  <link name="gripper_link" >
+    <visual>
+      <origin xyz="0 0 0" rpy="0 0 0" />
+      <geometry>
+	<sphere radius=".001"/>
+      </geometry>
+    </visual>
+  </link>
+  <!-- KINECT LINK ?? -->
+  <joint name="base_kinect_joint" type="fixed">
+    <origin xyz="0 0 0" rpy="0 0 0" />
+    <parent link="base_link"/>
+    <child link="kinect_link"/>
+  </joint>
+  <link name="kinect_link">
+    <visual>
+      <origin rpy="0 0 0" xyz=" 0 0 0 "/>
+      <geometry>
+	<sphere radius=".005"/>
+      </geometry>
+    </visual>
+  </link>
 </robot>

Commit message: Added tabletop model to URDF

File: clam_description/urdf/clam_urdf.xacro (robot description, xacro)
@@ -343,3 +343,18 @@
     </visual>
   </link>
+  <!-- TABLETOP MODEL -->
+  <joint name="tabletop_joint" type="fixed">
+    <origin xyz="0 0 0" rpy="0 0 0" />
+    <parent link="base_link"/>
+    <child link="tabletop_link"/>
+  </joint>
+  <link name="tabletop_link">
+    <visual>
+      <origin rpy="${.5*M_PI} 0 ${.5*M_PI}" xyz=" 0 0 -0.017"/>
+      <geometry>
+	<mesh filename="package://clam_description/stl/tabletop.STL" scale="1 1 1" />
+      </geometry>
+      <material name="White" />
+    </visual>
+  </link>
 </robot>

Commit message: Calibrated URDF to turn elbow_pitch_joint slightly

File: clam_description/urdf/clam_urdf.xacro (robot description, xacro)
@@ -115,5 +115,5 @@
     <parent link="elbow_roll_link"/>
     <child link="elbow_pitch_link"/>
-    <origin xyz="-0.035 0 0.0009" rpy="0 ${M_PI/2} 0" />
+    <origin xyz="-0.035 0 0.0009" rpy="0.05 ${M_PI/2} 0" />
     <axis xyz="1 0 0" />
     <limit effort="300" velocity="1" lower="-1.5953400194" upper="1.93281579274" />

Commit message: Renamed gripper_grip_controller to l_gripper_aft_controller because name inconsistency was causing issues with Dynamixel Hardware Interface

File: clam_description/urdf/clam_urdf.xacro (robot description, xacro)
@@ -35,8 +35,4 @@
       </geometry>
       </collision>>
-      <inertial>
-	<mass value="25" />
-	<inertia ixx="1.0" ixy ="0.0" ixz="0.0" iyy="1.0" iyz="0.0" izz="1.0" />
-      </inertial>
   </link>
   <joint name="shoulder_pan_joint" type="revolute">
@@ -115,5 +111,5 @@
     <parent link="elbow_roll_link"/>
     <child link="elbow_pitch_link"/>
-    <origin xyz="-0.035 0 0.0009" rpy="0.05 ${M_PI/2} 0" />
+    <origin xyz="-0.035 0 0.0009" rpy="0.065 ${M_PI/2} 0" />
     <axis xyz="1 0 0" />
     <limit effort="300" velocity="1" lower="-1.5953400194" upper="1.93281579274" />
@@ -197,9 +193,10 @@
       <origin xyz="0 0 0" rpy="0 0 0" />
       <geometry>
-	<mesh filename="package://clam_description/stl/gripper_grip_link.STL" scale="1 1 1" />
+	<mesh filename="package://clam_description/stl/l_gripper_aft_link.STL" scale="1 1 1" />
       </geometry>
       <material name="Orange" />
     </visual>
   </link>
+  <!--joint name="l_gripper_aft_joint" type="revolute"-->
   <joint name="l_gripper_aft_link_joint" type="revolute">
     <parent link="gripper_roll_link"/>
@@ -315,46 +312,3 @@
     </visual>
   </link>
-  <!-- FAKE CAMERA CALIBRATION POINT -->
-  <joint name="gripper_link_joint" type="fixed">
-    <origin xyz="0.012 -0.11 0.020" rpy="0 0 0" />
-    <parent link="l_gripper_pincher"/>
-    <child link="gripper_link" />
-  </joint>
-  <link name="gripper_link" >
-    <visual>
-      <origin xyz="0 0 0" rpy="0 0 0" />
-      <geometry>
-	<sphere radius=".001"/>
-      </geometry>
-    </visual>
-  </link>
-  <!-- KINECT LINK ?? -->
-  <joint name="base_kinect_joint" type="fixed">
-    <origin xyz="0 0 0" rpy="0 0 0" />
-    <parent link="base_link"/>
-    <child link="kinect_link"/>
-  </joint>
-  <link name="kinect_link">
-    <visual>
-      <origin rpy="0 0 0" xyz=" 0 0 0 "/>
-      <geometry>
-	<sphere radius=".005"/>
-      </geometry>
-    </visual>
-  </link>
-  <!-- TABLETOP MODEL -->
-  <joint name="tabletop_joint" type="fixed">
-    <origin xyz="0 0 0" rpy="0 0 0" />
-    <parent link="base_link"/>
-    <child link="tabletop_link"/>
-  </joint>
-  <link name="tabletop_link">
-    <visual>
-      <origin rpy="${.5*M_PI} 0 ${.5*M_PI}" xyz=" 0 0 -0.017"/>
-      <geometry>
-	<mesh filename="package://clam_description/stl/tabletop.STL" scale="1 1 1" />
-      </geometry>
-      <material name="White" />
-    </visual>
-  </link>
 </robot>

File: clam_description/urdf/materials.urdf.xacro (robot description, xacro)
@@ -16,4 +16,7 @@
         <color rgba="${255/255} ${108/255} ${10/255} 1.0"/>
     </material>
+    <material name="Brown">
+        <color rgba="${222/255} ${207/255} ${195/255} 1.0"/>
+    </material>
     <material name="Red">
         <color rgba="0.8 0.0 0.0 1.0"/>

Commit message: Fixing find and replace issues

File: clam_description/urdf/clam_urdf.xacro (robot description, xacro)
@@ -193,5 +193,5 @@
       <origin xyz="0 0 0" rpy="0 0 0" />
       <geometry>
-	<mesh filename="package://clam_description/stl/l_gripper_aft_link.STL" scale="1 1 1" />
+	<mesh filename="package://clam_description/stl/gripper_grip_link.STL" scale="1 1 1" />
       </geometry>
       <material name="Orange" />

Commit message: Calibrating arm model

File: clam_description/urdf/clam_urdf.xacro (robot description, xacro)
@@ -111,5 +111,5 @@
     <parent link="elbow_roll_link"/>
     <child link="elbow_pitch_link"/>
-    <origin xyz="-0.035 0 0.0009" rpy="0.065 ${M_PI/2} 0" />
+    <origin xyz="-0.035 0 0.0009" rpy="0.055 ${M_PI/2} 0" />
     <axis xyz="1 0 0" />
     <limit effort="300" velocity="1" lower="-1.5953400194" upper="1.93281579274" />
@@ -312,3 +312,33 @@
     </visual>
   </link>
+  <!-- TABLETOP MODEL -->
+  <joint name="tabletop_joint" type="fixed">
+    <origin xyz="0 0 0" rpy="0 0 0" />
+    <parent link="base_link"/>
+    <child link="tabletop_link"/>
+  </joint>
+  <link name="tabletop_link">
+    <visual>
+      <origin rpy="${.5*M_PI} 0 ${.5*M_PI}" xyz=" 0 0 -0.017"/>
+      <geometry>
+	<mesh filename="package://clam_description/stl/tabletop.STL" scale="1 1 1" />
+      </geometry>
+      <material name="Brown" />
+    </visual>
+  </link>
+  <!-- FAKE CAMERA CALIBRATION POINT -->
+  <joint name="gripper_link_joint" type="fixed">
+    <!--origin xyz="0.012 -0.11 0.020" rpy="0 0 0" /-->
+    <origin xyz="0.1795 0 0" rpy="0 0 0" />
+    <parent link="gripper_roll_link"/>
+    <child link="gripper_link" />
+  </joint>
+  <link name="gripper_link" >
+    <visual>
+      <origin xyz="0 0 0" rpy="0 0 0" />
+      <geometry>
+	<sphere radius=".001"/>
+      </geometry>
+    </visual>
+  </link>
 </robot>

Commit message: Calibrating URDF

File: clam_description/urdf/clam_urdf.xacro (robot description, xacro)
@@ -87,5 +87,5 @@
     <parent link="shoulder_pitch_link"/>
     <child link="elbow_roll_link"/>
-    <origin xyz="-0.001 0 0.121" rpy="${M_PI} ${M_PI/2} 0" />
+    <origin xyz="-0.002 0 0.1206" rpy="${M_PI} ${M_PI/2} 0" />
     <axis xyz="-1 0 0" />
     <limit effort="300" velocity="1" lower="-2.61799387799" upper="0.705631162427" />
@@ -111,5 +111,5 @@
     <parent link="elbow_roll_link"/>
     <child link="elbow_pitch_link"/>
-    <origin xyz="-0.035 0 0.0009" rpy="0.055 ${M_PI/2} 0" />
+    <origin xyz="-0.035 0 0.0" rpy="0.055 ${M_PI/2} 0" />
     <axis xyz="1 0 0" />
     <limit effort="300" velocity="1" lower="-1.5953400194" upper="1.93281579274" />

Commit message: Trying to fix wrist_pitch issue

File: clam_description/urdf/clam_urdf.xacro (robot description, xacro)
@@ -119,5 +119,5 @@
   <link name="elbow_pitch_link" >
     <visual>
-      <origin xyz="0.0 0 -${0.035*0}" rpy="${M_PI/2} 0 ${M_PI/2+M_PI}" />
+      <origin xyz="0.0 0 0" rpy="${M_PI/2} 0 ${M_PI/2+M_PI}" />
       <geometry>
 	<mesh filename="package://clam_description/stl/elbow_pitch_link.STL" scale="${M_SCALE}" />
@@ -126,5 +126,5 @@
     </visual>
     <collision>
-      <origin xyz="0.0 0 -${0.035*0}" rpy="${M_PI/2} 0 ${M_PI/2+M_PI}" />
+      <origin xyz="0.0 0 0" rpy="${M_PI/2} 0 ${M_PI/2+M_PI}" />
       <geometry>
 	<mesh filename="package://clam_description/stl/elbow_pitch_link_simple.STL" scale="${M_SCALE}" />

Commit message: Calibrating urdf

File: clam_description/urdf/clam_urdf.xacro (robot description, xacro)
@@ -63,5 +63,5 @@
     <parent link="shoulder_pan_link"/>
     <child link="shoulder_pitch_link"/>
-    <origin xyz="-0.041 0.0 0.0" rpy="-${M_PI/2} 0 ${M_PI/2}" />
+    <origin xyz="-0.041 0.0021 0.0" rpy="-${M_PI/2} 0 ${M_PI/2}" />
     <axis xyz="1 0 0" />
     <limit effort="300" velocity="1" lower="-1.19962513147" upper="1.89994105047" />
@@ -135,5 +135,5 @@
     <parent link="elbow_pitch_link"/>
     <child link="wrist_roll_link"/>
-    <origin xyz="0.0 0.008 -.248" rpy="0 ${M_PI/2} ${M_PI}" />
+    <origin xyz="0.0 0.0081 -.248" rpy="0 ${M_PI/2} ${M_PI}" />
     <axis xyz="1 0 0" />
     <limit effort="300" velocity="1" lower="-2.61799387799" upper="2.6128806087" />
@@ -159,5 +159,5 @@
     <parent link="wrist_roll_link"/>
     <child link="wrist_pitch_link"/>
-    <origin xyz="0.0 0.0 ${1*0.002}" rpy="0 ${M_PI/2} 0" />
+    <origin xyz="0.0 0.0 0.0001" rpy="0 ${M_PI/2} 0" />
     <axis xyz="1 0 0" />
     <limit effort="300" velocity="1" lower="-1.5953400194" upper="1.98394848567" />
@@ -183,5 +183,5 @@
     <parent link="wrist_pitch_link"/>
     <child link="gripper_roll_link"/>
-    <origin xyz="0 0 0.08" rpy="${1.5*M_PI} -${.5*M_PI} 0" />
+    <origin xyz="0 0 0.08065" rpy="${1.5*M_PI} -${.5*M_PI} 0" />
     <axis xyz="1 0 0" />
     <limit effort="300" velocity="1" lower="-2.61799387799" upper="2.6128806087" />
