Commit message: Finished tweaking URDF, updated ClamArm Technical Diagram

File: clam_description/urdf/clam_urdf.xacro (robot description, xacro)
@@ -183,5 +183,5 @@
     <parent link="wrist_pitch_link"/>
     <child link="gripper_roll_link"/>
-    <origin xyz="0 0 0.08065" rpy="${1.5*M_PI} -${.5*M_PI} 0" />
+    <origin xyz="0 0 0.080" rpy="${1.5*M_PI} -${.5*M_PI} 0" />
     <axis xyz="1 0 0" />
     <limit effort="300" velocity="1" lower="-2.61799387799" upper="2.6128806087" />
@@ -202,5 +202,5 @@
     <parent link="gripper_roll_link"/>
     <child link="l_gripper_aft_link"/>
-    <origin xyz="0.025 ${-0.0275+.040} 0" rpy="${1.04*M_PI} ${M_PI/2} ${34.58*M_PI/180}" />
+    <origin xyz="0.026 .017 0" rpy="${1.04*M_PI} ${M_PI/2} ${34.58*M_PI/180}" />
     <axis xyz="1 0 0" />
     <limit effort="300" velocity="1" lower="${0*M_PI/180}" upper="${-53*M_PI/180}" />
@@ -220,5 +220,5 @@
     <parent link="gripper_roll_link"/>
     <child link="r_gripper_aft_link"/>
-    <origin xyz="0.025 ${-0.0561+.040}  0" rpy="${1.345*M_PI} ${M_PI/2} ${34.58*M_PI/180}" />
+    <origin xyz="0.026 -0.011  0" rpy="${1.345*M_PI} ${M_PI/2} ${34.58*M_PI/180}" />
     <axis xyz="1 0 0" />
     <limit effort="300" velocity="1" lower="-3.14" upper="3.14" />
@@ -239,5 +239,5 @@
     <parent link="gripper_roll_link"/>
     <child link="l_gripper_fwd_link"/>
-    <origin xyz="0.05 ${-0.037+.040} 0.007" rpy="${M_PI*(1+.04)} ${M_PI/2} ${214.58*M_PI/180}" />
+    <origin xyz="0.05 0.008 0.007" rpy="${M_PI*(1+.04)} ${M_PI/2} ${214.58*M_PI/180}" />
     <axis xyz="1 0 0" />
     <limit effort="300" velocity="1" lower="0" upper="1.57" />
@@ -258,5 +258,5 @@
     <parent link="gripper_roll_link"/>
     <child link="r_gripper_fwd_link"/>
-    <origin xyz="0.05 ${-0.047+.040} 0.007" rpy="${M_PI*(1-.04)} ${M_PI/2} ${145.42*M_PI/180}" />
+    <origin xyz="0.05 -0.0014 0.007" rpy="${M_PI*(1-.04)} ${M_PI/2} ${145.42*M_PI/180}" />
     <axis xyz="1 0 0" />
     <limit effort="300" velocity="1" lower="-1.57" upper="0" />
@@ -277,5 +277,5 @@
     <parent link="l_gripper_aft_link"/>
     <child link="l_gripper_pincher"/>
-    <origin xyz="-0.0032 0 -0.0508" rpy="${203.27*M_PI/180-.312*M_PI} 0 0" />
+    <origin xyz="-0.0032 0 -0.0508" rpy="${203.27*M_PI/180-.3150*M_PI} 0 0" />
     <axis xyz="1 0 0" />
     <limit effort="300" velocity="1" lower="-1.57" upper="1.57" />
@@ -296,5 +296,5 @@
     <parent link="r_gripper_aft_link"/>
     <child link="r_gripper_pincher"/>
-    <origin xyz="0 0 -0.0508" rpy="${23.27*M_PI/180-.312*M_PI} ${M_PI} 0" />
+    <origin xyz="0 0 -0.0508" rpy="${23.27*M_PI/180-.3150*M_PI} ${M_PI} 0" />
     <axis xyz="1 0 0" />
     <limit effort="300" velocity="1" lower="0" upper="1.57" />

Commit message: Integrated clam_kinect_arm_calibration package from turtlebot. Finished calibrating kinect.

File: clam_description/urdf/clam_urdf.xacro (robot description, xacro)
@@ -199,5 +199,5 @@
   </link>
   <!--joint name="l_gripper_aft_joint" type="revolute"-->
-  <joint name="l_gripper_aft_link_joint" type="revolute">
+  <joint name="l_gripper_aft_joint" type="revolute">
     <parent link="gripper_roll_link"/>
     <child link="l_gripper_aft_link"/>
@@ -223,5 +223,5 @@
     <axis xyz="1 0 0" />
     <limit effort="300" velocity="1" lower="-3.14" upper="3.14" />
-    <mimic joint="l_gripper_aft_link_joint" multiplier="-1.0" offset="0.0" />
+    <mimic joint="l_gripper_aft_joint" multiplier="-1.0" offset="0.0" />
     <dynamics damping="50" friction="1"/>
   </joint>
@@ -242,5 +242,5 @@
     <axis xyz="1 0 0" />
     <limit effort="300" velocity="1" lower="0" upper="1.57" />
-    <mimic joint="l_gripper_aft_link_joint" multiplier="1.0" offset="0" />
+    <mimic joint="l_gripper_aft_joint" multiplier="1.0" offset="0" />
     <dynamics damping="50" friction="1"/>
   </joint>
@@ -261,5 +261,5 @@
     <axis xyz="1 0 0" />
     <limit effort="300" velocity="1" lower="-1.57" upper="0" />
-    <mimic joint="l_gripper_aft_link_joint" multiplier="-1.0" offset="0" />
+    <mimic joint="l_gripper_aft_joint" multiplier="-1.0" offset="0" />
     <dynamics damping="50" friction="1"/>
   </joint>
@@ -280,5 +280,5 @@
     <axis xyz="1 0 0" />
     <limit effort="300" velocity="1" lower="-1.57" upper="1.57" />
-    <mimic joint="l_gripper_aft_link_joint" multiplier="-1.0" offset="0" />
+    <mimic joint="l_gripper_aft_joint" multiplier="-1.0" offset="0" />
     <dynamics damping="50" friction="1"/>
   </joint>
@@ -299,5 +299,5 @@
     <axis xyz="1 0 0" />
     <limit effort="300" velocity="1" lower="0" upper="1.57" />
-    <mimic joint="l_gripper_aft_link_joint" multiplier="-1.0" offset="0" />
+    <mimic joint="l_gripper_aft_joint" multiplier="-1.0" offset="0" />
     <dynamics damping="50" friction="1"/>
   </joint>
@@ -342,3 +342,17 @@
     </visual>
   </link>
+  <!-- KINECT LINK ?? -->
+  <joint name="base_kinect_joint" type="fixed">
+    <origin xyz="0 0 0" rpy="0 0 0" />
+    <parent link="base_link"/>
+    <child link="kinect_link"/>
+  </joint>
+  <link name="kinect_link">
+    <visual>
+      <origin rpy="0 0 0" xyz=" 0 0 0 "/>
+      <geometry>
+	<sphere radius=".005"/>
+      </geometry>
+    </visual>
+  </link>
 </robot>

Commit message: Trying to fix the warning message about joint states not being published Updated autostart scripts

File: clam_description/urdf/clam_urdf.xacro (robot description, xacro)
@@ -198,5 +198,4 @@
     </visual>
   </link>
-  <!--joint name="l_gripper_aft_joint" type="revolute"-->
   <joint name="l_gripper_aft_joint" type="revolute">
     <parent link="gripper_roll_link"/>
@@ -312,47 +311,3 @@
     </visual>
   </link>
-  <!-- TABLETOP MODEL -->
-  <joint name="tabletop_joint" type="fixed">
-    <origin xyz="0 0 0" rpy="0 0 0" />
-    <parent link="base_link"/>
-    <child link="tabletop_link"/>
-  </joint>
-  <link name="tabletop_link">
-    <visual>
-      <origin rpy="${.5*M_PI} 0 ${.5*M_PI}" xyz=" 0 0 -0.017"/>
-      <geometry>
-	<mesh filename="package://clam_description/stl/tabletop.STL" scale="1 1 1" />
-      </geometry>
-      <material name="Brown" />
-    </visual>
-  </link>
-  <!-- FAKE CAMERA CALIBRATION POINT -->
-  <joint name="gripper_link_joint" type="fixed">
-    <!--origin xyz="0.012 -0.11 0.020" rpy="0 0 0" /-->
-    <origin xyz="0.1795 0 0" rpy="0 0 0" />
-    <parent link="gripper_roll_link"/>
-    <child link="gripper_link" />
-  </joint>
-  <link name="gripper_link" >
-    <visual>
-      <origin xyz="0 0 0" rpy="0 0 0" />
-      <geometry>
-	<sphere radius=".001"/>
-      </geometry>
-    </visual>
-  </link>
-  <!-- KINECT LINK ?? -->
-  <joint name="base_kinect_joint" type="fixed">
-    <origin xyz="0 0 0" rpy="0 0 0" />
-    <parent link="base_link"/>
-    <child link="kinect_link"/>
-  </joint>
-  <link name="kinect_link">
-    <visual>
-      <origin rpy="0 0 0" xyz=" 0 0 0 "/>
-      <geometry>
-	<sphere radius=".005"/>
-      </geometry>
-    </visual>
-  </link>
 </robot>

Commit message: Renamed package: clam_kinect_arm_calibration -> clam_openni_vision Also handles launching vision components now

File: clam_description/urdf/clam_urdf.xacro (robot description, xacro)
@@ -311,3 +311,33 @@
     </visual>
   </link>
+  <!-- TABLETOP MODEL -->
+  <joint name="tabletop_joint" type="fixed">
+    <origin xyz="0 0 0" rpy="0 0 0" />
+    <parent link="base_link"/>
+    <child link="tabletop_link"/>
+  </joint>
+  <link name="tabletop_link">
+    <visual>
+      <origin rpy="${.5*M_PI} 0 ${.5*M_PI}" xyz=" 0 0 -0.017"/>
+      <geometry>
+	<mesh filename="package://clam_description/stl/tabletop.STL" scale="1 1 1" />
+      </geometry>
+      <material name="Brown" />
+    </visual>
+  </link>
+  <!-- FAKE CAMERA CALIBRATION POINT -->
+  <joint name="gripper_link_joint" type="fixed">
+    <!--origin xyz="0.012 -0.11 0.020" rpy="0 0 0" /-->
+    <origin xyz="0.1795 0 0" rpy="0 0 0" />
+    <parent link="gripper_roll_link"/>
+    <child link="gripper_link" />
+  </joint>
+  <link name="gripper_link" >
+    <visual>
+      <origin xyz="0 0 0" rpy="0 0 0" />
+      <geometry>
+	<sphere radius=".001"/>
+      </geometry>
+    </visual>
+  </link>
 </robot>

Commit message: Fixes for the arm_navigation grasping pipeline

File: clam_description/urdf/clam_urdf.xacro (robot description, xacro)
@@ -326,5 +326,5 @@
     </visual>
   </link>
-  <!-- FAKE CAMERA CALIBRATION POINT -->
+  <!-- FAKE CAMERA CALIBRATION POINT AT GRIPPER TIP  -->
   <joint name="gripper_link_joint" type="fixed">
     <!--origin xyz="0.012 -0.11 0.020" rpy="0 0 0" /-->
@@ -341,3 +341,17 @@
     </visual>
   </link>
+  <!-- KINECT LINK - Needed? -->
+  <!--joint name="base_kinect_joint" type="fixed">
+    <origin xyz="0.769541 -0.0539292 0.836631" rpy="0 0 0" />
+    <parent link="base_link"/>
+    <child link="camera_link"/>
+  </joint>
+  <link name="camera_link">
+    <visual>
+      <origin rpy="0 0 0" xyz=" 0 0 0 "/>
+      <geometry>
+	<sphere radius=".005"/>
+      </geometry>
+    </visual>
+  </link-->
 </robot>

Commit message: Added new published plane feature to block detection

File: clam_description/urdf/clam_urdf.xacro (robot description, xacro)
@@ -341,6 +341,7 @@
     </visual>
   </link>
-  <!-- KINECT LINK - Needed? -->
-  <!--joint name="base_kinect_joint" type="fixed">
+  <!-- KINECT LINK - Not Needed! -->
+<!--
+  <joint name="base_kinect_joint" type="fixed">
     <origin xyz="0.769541 -0.0539292 0.836631" rpy="0 0 0" />
     <parent link="base_link"/>
@@ -354,4 +355,5 @@
       </geometry>
     </visual>
-  </link-->
+  </link>
+-->
 </robot>

Commit message: Renamed urdf file, restructured launch files

File: clam_description/urdf/clam_urdf.xacro (robot description, xacro)
@@ -312,5 +312,5 @@
   </link>
   <!-- TABLETOP MODEL -->
-  <joint name="tabletop_joint" type="fixed">
+  <!--joint name="tabletop_joint" type="fixed">
     <origin xyz="0 0 0" rpy="0 0 0" />
     <parent link="base_link"/>
@@ -325,5 +325,5 @@
       <material name="Brown" />
     </visual>
-  </link>
+  </link-->
   <!-- FAKE CAMERA CALIBRATION POINT AT GRIPPER TIP  -->
   <joint name="gripper_link_joint" type="fixed">

File: clam_description/urdf/clam_urdf_generated.urdf (robot description, URDF)
Before this commit: robot clam, 16 links, 15 joints
Links:
- removed link tabletop_link
Joints:
- removed joint tabletop_joint
